File: pcb/pcb.kicad_pcb (KiCad board)
At the start: 2 copper layers, 21 x 51 mm, 33 parts, among them J1 USB_C_Receptacle_USB2.0_14P, J2 Conn_01x20, J3 Conn_01x20, J4 Conn_01x03, SW1 SW_Push, U1 RP2040, U2 MCP1700x-330xxTT, U3 W25Q128JVS, Y1 Crystal_GND24

Commit message: update pcb
Parts:
- C15, C16: value 15pF -> 33pF
- U3: value W25Q128JVS -> W25Q16JVZPIQ TR; footprint Package_SO:SOIC-8_5.3x5.3mm_P1.27mm -> W25Q16JVUXIQ_TR:IC_W25Q16JVUXIQ_TR
- Y1: value Crystal_GND24 -> 12 MHz
- moved R1 83.5 mm to (206.5, 67.7)
- moved C6 79.7 mm to (208.0, 86.2)
- moved R2 79.7 mm to (201.5, 67.6), turned to 180 degrees
- moved C2 79.7 mm to (208.8, 90.2)
- moved R4 78.6 mm to (204.8, 83.3), turned to -90 degrees
- moved C5 78.6 mm to (206.8, 84.3), turned to 45 degrees
- moved R3 77.1 mm to (203.8, 83.3), turned to -90 degrees
- moved R6 77.1 mm to (200.8, 80.4), turned to 180 degrees
- moved C1 76.8 mm to (205.8, 95.0), turned to -90 degrees
- moved C8 76.5 mm to (207.6, 85.0), turned to 90 degrees
- moved R5 76.2 mm to (204.5, 94.1), turned to 180 degrees
- moved R7 76.0 mm to (198.7, 80.2), turned to 90 degrees
- moved C12 76.0 mm to (206.0, 83.8), turned to 90 degrees
- moved C3 75.7 mm to (203.9, 81.2), turned to 90 degrees
- moved C4 75.3 mm to (203.2, 80.9), turned to 90 degrees
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Connections:
- J3 pad 1: GPIO16 -> VBUS
- J3 pad 10: RUN -> GPIO23
- J3 pad 11: GPIO23 -> RUN
- J3 pad 12: GPIO24 -> GPIO22
- J3 pad 14: GPIO25 -> GPIO21
- J3 pad 15: GPIO26_ADC0 -> GPIO20
- J3 pad 16: +3V3 -> GPIO19
- J3 pad 17: GPIO27_ADC1 -> GPIO18
- J3 pad 19: GPIO28_ADC2 -> GPIO17
- J3 pad 2: GPIO17 -> GPIO28_ADC2
- J3 pad 20: VBUS -> GPIO16
- J3 pad 4: GPIO18 -> GPIO27_ADC1
- J3 pad 5: GPIO19 -> +3V3
- J3 pad 6: GPIO20 -> GPIO26_ADC0
- J3 pad 7: GPIO21 -> GPIO25
- J3 pad 9: GPIO22 -> GPIO24
Routing:
- net +3V3: track 0.00 -> 82.5 mm, vias 0 -> 5
- net GND: track 0.00 -> 44.1 mm, vias 0 -> 14
- net +1V1: track 0.00 -> 43.8 mm, vias 0 -> 4
- net GPIO0: track 0.00 -> 28.5 mm, vias 0 -> 2
- net GPIO1: track 0.00 -> 27.9 mm, vias 0 -> 2
- net GPIO28_ADC2: track 0.00 -> 27.3 mm
- net GPIO27_ADC1: track 0.00 -> 22.7 mm
- net USB_D+: track 0.00 -> 22.2 mm
- net USB_D-: track 0.00 -> 22.2 mm
- net GPIO2: track 0.00 -> 22.1 mm
- net GPIO16: track 0.00 -> 21.5 mm, vias 0 -> 2
- net GPIO15: track 0.00 -> 21.2 mm
- net SWCLK: track 0.00 -> 21.1 mm, vias 0 -> 2
- net VBUS: track 0.00 -> 20.5 mm
- net GPIO3: track 0.00 -> 20.1 mm
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- added copper zone on B.Cu, net GND
- added copper zone on F.Cu, net GND
