File: pcb/pcb.kicad_pcb (KiCad board)
At the start: 2 copper layers, 21 x 51 mm, 33 parts, among them J1 USB_C_Receptacle_USB2.0_14P, J2 Conn_01x20, J3 Conn_01x20, J4 Conn_01x03, SW1 SW_Push, U1 RP2040, U2 MCP1700x-330xxTT, U3 W25Q16JVZPIQ TR, Y1 12 MHz

Commit message: update pcb, readme, BOM
Parts:
- added C18: 0.1uF, Capacitor_SMD:C_01005_0402Metric, F.Cu at (199.4, 98.9)
- added R8: 4.7K, Resistor_SMD:R_0402_1005Metric, F.Cu at (201.0, 98.8)
- added R9: 4.7K, Resistor_SMD:R_0402_1005Metric, F.Cu at (202.3, 100.2)
- added U4: TSL25911FN, OptoDevice:AMS_TSL25911FN, F.Cu at (200.2, 100.7)
- C10: value C -> 1uF
- C11, C12: value C -> 0.1uF
- moved C16 0.52 mm to (206.3, 96.6)
Routing:
- net GND: track 44.1 -> 81.7 mm, vias 14 -> 19
- net +3V3: track 82.5 -> 101.7 mm, vias 5 -> 9
- net GPIO11: track 8.42 -> 26.3 mm, vias 0 -> 4
- net GPIO10: track 6.56 -> 20.9 mm, vias 0 -> 4
- net GPIO12: track 10.3 -> 19.1 mm, vias 0 -> 2
- net GPIO7: track 10.4 -> 17.7 mm
- net SWCLK: track 21.1 -> 23.8 mm
- net Net-(C16-Pad2): track 3.35 -> 3.90 mm
- net (no net): track 0.00 -> 0.25 mm, vias 0 -> 13
