File: pcb/pcb.kicad_pcb (KiCad board)
At the start: 2 copper layers, 21 x 51 mm, 37 parts, among them J1 USB_C_Receptacle_USB2.0_14P, J2 Conn_01x20, J3 Conn_01x20, J4 Conn_01x03, SW1 SW_Push, U1 RP2040, U2 MCP1700x-330xxTT, U3 W25Q16JVZPIQ TR, U4 TSL25911FN, Y1 12 MHz

Commit message: update README, silkscreen
Other:
- board text added: "nani board"
Changed lines of the file:
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@@
 		(layer "Edge.Cuts")
+	)
+	(gr_text "nani board\n"
+		(at 209.79 108.64 90)
+		(layer "F.SilkS")
+		(effects
+			(font
+				(size 1 1)
+				(thickness 0.1)
+			)
+			(justify left bottom)
+		)
 	)
 	(segment
