File: pcb/pcb.kicad_sch (KiCad schematic)
At the start: 33 parts, among them J1 USB_C_Receptacle_USB2.0_14P, J2 Conn_01x20, J3 Conn_01x20, J4 Conn_01x03, SW1 SW_Push, U1 RP2040, U2 MCP1700x-330xxTT, U3 W25Q128JVS, Y1 Crystal_GND24

Commit message: update pcb
Parts:
- C15, C16: value 15pF -> 33pF
- U3: value W25Q128JVS -> W25Q16JVZPIQ TR; footprint Package_SO:SOIC-8_5.3x5.3mm_P1.27mm -> W25Q16JVUXIQ_TR:IC_W25Q16JVUXIQ_TR
- Y1: value Crystal_GND24 -> 12 MHz
Connections:
- net +3V3: now also J3.5 (Pin_5); no longer J3.16 (Pin_16)
- net GPIO16: now also J3.20 (Pin_20); no longer J3.1 (Pin_1)
- net GPIO17: now also J3.19 (Pin_19); no longer J3.2 (Pin_2)
- net GPIO18: now also J3.17 (Pin_17); no longer J3.4 (Pin_4)
- net GPIO19: now also J3.16 (Pin_16); no longer J3.5 (Pin_5)
- net GPIO20: now also J3.15 (Pin_15); no longer J3.6 (Pin_6)
- net GPIO21: now also J3.14 (Pin_14); no longer J3.7 (Pin_7)
- net GPIO22: now also J3.12 (Pin_12); no longer J3.9 (Pin_9)
- net GPIO23: now also J3.10 (Pin_10); no longer J3.11 (Pin_11)
- net GPIO24: now also J3.9 (Pin_9); no longer J3.12 (Pin_12)
- net GPIO25: now also J3.7 (Pin_7); no longer J3.14 (Pin_14)
- net GPIO26_ADC0: now also J3.6 (Pin_6); no longer J3.15 (Pin_15)
- net GPIO27_ADC1: now also J3.4 (Pin_4); no longer J3.17 (Pin_17)
- net GPIO28_ADC2: now also J3.2 (Pin_2); no longer J3.19 (Pin_19)
- net RUN: now also J3.11 (Pin_11); no longer J3.10 (Pin_10)
- net VBUS: now also J3.1 (Pin_1); no longer J3.20 (Pin_20)
Other:
- moved on the sheet: J3
Changed lines of the file:
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@@
 	(wire
 		(pts
-			(xy 67.31 116.84) (xy 71.12 116.84)
-		)
-		(stroke
-			(width 0)
-			(type default)
-		)
-	)
-	(wire
-		(pts
 			(xy 33.02 129.54) (xy 36.83 129.54)
 		)
@@
 	(wire
 		(pts
+			(xy 67.31 137.16) (xy 71.12 137.16)
+		)
+		(stroke
+			(width 0)
+			(type default)
+		)
+	)
+	(wire
+		(pts
 			(xy 256.54 97.79) (xy 260.35 97.79)
 		)
@@
 	(wire
 		(pts
-			(xy 67.31 137.16) (xy 71.12 137.16)
-		)
-		(stroke
-			(width 0)
-			(type default)
-		)
-	)
-	(wire
-		(pts
 			(xy 77.47 31.75) (xy 77.47 33.02)
 		)
@@
 	(wire
 		(pts
-			(xy 67.31 111.76) (xy 71.12 111.76)
-		)
-		(stroke
-			(width 0)
-			(type default)
-		)
-	)
-	(wire
-		(pts
 			(xy 48.26 36.83) (xy 48.26 38.1)
 		)
@@
 	(wire
 		(pts
+			(xy 67.31 111.76) (xy 71.12 111.76)
+		)
+		(stroke
+			(width 0)
+			(type default)
+		)
+	)
+	(wire
+		(pts
 			(xy 33.02 139.7) (xy 36.83 139.7)
 		)
@@
 	(wire
 		(pts
-			(xy 241.3 29.21) (xy 241.3 30.48)
+			(xy 67.31 104.14) (xy 71.12 104.14)
 		)
 		(stroke
@@
 	(wire
 		(pts
-			(xy 48.26 24.13) (xy 57.15 24.13)
+			(xy 241.3 29.21) (xy 241.3 30.48)
 		)
 		(stroke
@@
 	(wire
 		(pts
-			(xy 177.8 139.7) (xy 180.34 139.7)
+			(xy 48.26 24.13) (xy 57.15 24.13)
 		)
 		(stroke
@@
 	(wire
 		(pts
-			(xy 67.31 93.98) (xy 71.12 93.98)
+			(xy 177.8 139.7) (xy 180.34 139.7)
 		)
 		(stroke
@@
 	(wire
 		(pts
+			(xy 67.31 116.84) (xy 71.12 116.84)
+		)
+		(stroke
+			(width 0)
+			(type default)
+		)
+	)
+	(wire
+		(pts
 			(xy 33.02 116.84) (xy 36.83 116.84)
 		)
@@
 	(wire
 		(pts
-			(xy 67.31 104.14) (xy 71.12 104.14)
+			(xy 67.31 93.98) (xy 71.12 93.98)
 		)
 		(stroke
@@
 			)
 		)
-		(property "Value" "Crystal_GND24"
+		(property "Value" "12 MHz"
 			(at 252.476 90.17 90)
 			(effects
@@
 			)
 		)
-		(property "Value" "15pF"
+		(property "Value" "33pF"
 			(at 223.52 88.138 90)
 			(effects
@@
 	(symbol
 		(lib_id "Connector_Generic:Conn_01x20")
-		(at 62.23 116.84 180)
+		(at 62.23 114.3 0)
+		(mirror y)
 		(unit 1)
 		(exclude_from_sim no)
@@
 		(on_board yes)
 		(dnp no)
-		(fields_autoplaced yes)
 		(property "Reference" "J3"
-			(at 62.23 85.09 0)
+			(at 59.69 114.2999 0)
 			(effects
 				(font
 					(size 1.27 1.27)
 				)
+				(justify left)
 			)
 		)
 		(property "Value" "Conn_01x20"
-			(at 62.23 87.63 0)
+			(at 59.69 116.8399 0)
 			(effects
 				(font
 					(size 1.27 1.27)
 				)
+				(justify left)
 			)
 		)
 		(property "Footprint" "Connector_PinHeader_2.54mm:PinHeader_1x20_P2.54mm_Vertical"
-			(at 62.23 116.84 0)
+			(at 62.23 114.3 0)
 			(effects
 				(font
@@
 		)
 		(property "Datasheet" "~"
-			(at 62.23 116.84 0)
+			(at 62.23 114.3 0)
 			(effects
 				(font
@@
 		)
 		(property "Description" "Generic connector, single row, 01x20, script generated (kicad-library-utils/schlib/autogen/connector/)"
-			(at 62.23 116.84 0)
+			(at 62.23 114.3 0)
 			(effects
 				(font
@@
 			)
 		)
-		(property "Value" "W25Q128JVS"
+		(property "Value" "W25Q16JVZPIQ TR"
 			(at 269.24 48.2599 0)
 			(effects
@@
 			)
 		)
-		(property "Footprint" "Package_SO:SOIC-8_5.3x5.3mm_P1.27mm"
+		(property "Footprint" "W25Q16JVUXIQ_TR:IC_W25Q16JVUXIQ_TR"
 			(at 257.81 24.13 0)
 			(effects
@@
 			)
 		)
-		(property "Value" "15pF"
+		(property "Value" "33pF"
 			(at 222.25 99.314 90)
 			(effects
