File: pcb/pcb.kicad_sch (KiCad schematic)
At the start: 33 parts, among them J1 USB_C_Receptacle_USB2.0_14P, J2 Conn_01x20, J3 Conn_01x20, J4 Conn_01x03, SW1 SW_Push, U1 RP2040, U2 MCP1700x-330xxTT, U3 W25Q16JVZPIQ TR, Y1 12 MHz

Commit message: update pcb, readme, BOM
Parts:
- added C18: 0.1uF, Capacitor_SMD:C_01005_0402Metric, symbol Device:C
- added R8, R9: 4.7K, Resistor_SMD:R_0402_1005Metric, symbol Device:R
- added U4: TSL25911FN, OptoDevice:AMS_TSL25911FN, symbol Sensor_Optical:TSL25911FN
- C10: value C -> 1uF
- C11, C12: value C -> 0.1uF
Connections:
- net +3V3: now also C18.2, R8.1, R9.2, U4.5 (VDD)
- net GND: now also C18.1, U4.3 (GND)
- net GPIO10: now also R8.2, U4.6 (SDA)
- net GPIO11: now also R9.1, U4.1 (SCL)
- net GPIO12: now also U4.2 (INT)
